File: hardware/zegarek/zegarek.kicad_pcb (KiCad board)
At the start: 4 copper layers, 206.5 x 93 mm, 105 parts, among them J1 Barrel_Jack_MountingPin, J2 Conn_01x02, J3 Conn_01x02, J4 Conn_01x04, P1 USB_C_Plug_USB2.0, Q1 IRF740, SW1 SW_Push, SW2 SW_Push, SW3 SW_Push, SW4 SW_Push, U1 DI78L3.3UAB, U2 MC34063AD, U3 L7805ACV, U4 STM32F091RCTx, U5 CH340C, U6 74141, U7 74141, U8 74141, U9 74141, Y1 32.768kHz

Commit message: added kicad postprod jobset and postprod files
Parts:
- Q1, U3: footprint Package_TO_SOT_THT:TO-220-3_Horizontal_TabDown -> Package_TO_SOT_THT:TO-220-3_Horizontal_TabUp
- moved C26 24.5 mm to (132.8, 84.3)
- moved IN1 24.5 mm to (78.3, 135.2)
- moved R12 24.5 mm to (48.2, 87.1)
- moved BZ1 24.5 mm to (204.0, 64.6)
- moved C1 24.5 mm to (241.0, 111.1)
- moved C10 24.5 mm to (51.5, 97.6)
- moved C11 24.5 mm to (160.0, 53.2)
- moved C14 24.5 mm to (150.2, 79.6)
- moved C2 24.5 mm to (241.0, 121.1)
- moved C20 24.5 mm to (148.7, 69.1)
- moved C21 24.5 mm to (162.2, 78.4)
- moved C24 24.5 mm to (106.0, 73.1)
- moved C25 24.5 mm to (104.5, 84.1)
- moved C27 24.5 mm to (164.5, 84.6)
- moved C28 24.5 mm to (205.0, 84.6)
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Routing:
- net GND: track 126.4 -> 108.8 mm, vias 35 -> 133
- net /MCU/D+: track 4.59 -> 10.1 mm
- net /MCU/D-: track 4.59 -> 10.1 mm
- net Net-(U5-VCC): track 20.3 -> 24.6 mm
- net +3V3: track 354.3 -> 358.5 mm
- net +12V: track 78.0 -> 78.6 mm
- removed copper zone on B.Cu, net (none)
Other:
- outline, holes or cut-outs redrawn
- board text added: "3V3"
- board text added: "BOOT"
- board text added: "DEBUG"
- board text added: "DEBUG RX"
- board text added: "DEBUG TX"
- board text added: "GND"
- board text added: "PWR IN"
- board text added: "SWD"
- board text added: "TCK"
- board text added: "TMS"
- board text added: "zegarek v0"

Commit message: jlc generated bom and grb+drill
Parts:
- C17, C18: footprint Capacitor_SMD:C_1206_3216Metric_Pad1.33x1.80mm_HandSolder -> Capacitor_SMD:C_0603_1608Metric_Pad1.08x0.95mm_HandSolder
- R2: footprint Capacitor_SMD:C_0603_1608Metric_Pad1.08x0.95mm_HandSolder -> Resistor_SMD:R_0603_1608Metric_Pad0.98x0.95mm_HandSolder
- moved C18 0.52 mm to (145.2, 63.8)
- moved C17 0.44 mm to (145.2, 68.5)
Routing:
- net GND: track 108.8 -> 110.4 mm, vias 133 -> 134
Other:
- board text added: "x"
- board text removed: "0,3000 mm"
