File: hardware/zegarek/zegarek.kicad_pcb (KiCad board)
At the start: 4 copper layers, 100 x 100 mm, 106 parts, among them J1 Barrel_Jack_MountingPin, J2 Conn_01x02, J3 Conn_01x02, J4 Conn_01x04, M1 74141DIP16, M2 74141DIP16, M3 74141DIP16, M4 74141DIP16, Q1 IRF740, SW1 SW_Push, SW2 SW_Push, SW3 SW_Push, SW4 SW_Push, U1 DI78L3.3UAB, U2 MC34063AD, U3 L7805ACV, U4 STM32F091RCTx, U5 SN74LVC8T245, U6 SN74LVC8T245, Y1 32.768kHz

Commit message: reqenerating postprod
Parts:
- added C24: 100u, Capacitor_SMD:C_1206_3216Metric_Pad1.33x1.80mm_HandSolder, B.Cu at (76.8, 82.8)
- added F1: Fuse, Fuse:Fuse_1812_4532Metric_Pad1.30x3.40mm_HandSolder, B.Cu at (61.6, 63.6)
- added R43: 10k, Resistor_SMD:R_0603_1608Metric_Pad0.98x0.95mm_HandSolder, F.Cu at (98.4, 86.5)
- added R44: 1k, Resistor_SMD:R_0603_1608Metric_Pad0.98x0.95mm_HandSolder, F.Cu at (112.3, 50.5)
- added R46: 10k, Resistor_SMD:R_0603_1608Metric_Pad0.98x0.95mm_HandSolder, F.Cu at (110.6, 89.9)
- added R47: 1k, Resistor_SMD:R_0603_1608Metric_Pad0.98x0.95mm_HandSolder, F.Cu at (110.8, 50.6)
- added RN1: 10k, Resistor_SMD:R_Array_Convex_2x0606, F.Cu at (109.9, 83.3)
- added RN2: 10k, Resistor_SMD:R_Array_Convex_2x0606, F.Cu at (97.1, 82.7)
- C17, C18: value 4.3p -> 4.3p?
- R15, R4, R5, R6: value 4k7 -> 10k
- R31, R32, R41, R42: value 15k -> 56k; footprint Resistor_SMD:R_0603_1608Metric_Pad0.98x0.95mm_HandSolder -> Resistor_SMD:R_1206_3216Metric_Pad1.30x1.75mm_HandSolder
- moved SW4 5.96 mm to (140.9, 62.9), turned to 0 degrees
- moved R15 3.74 mm to (137.0, 64.4), turned to 90 degrees
- moved R13 2.95 mm to (137.2, 60.9), turned to 90 degrees
- moved J1 2.68 mm to (61.5, 58.8)
- moved C13 2.55 mm to (128.0, 63.1), turned to 45 degrees
- moved C8 0.70 mm to (79.2, 83.8)
- moved U3 0.60 mm to (81.7, 82.3)
- moved C9 0.40 mm to (86.6, 86.9)
- moved C6 0.19 mm to (58.8, 68.1)
Connections:
- J1 pad 1: +12V -> Net-(F1-Pad1)
- U4 pad 24: unconnected-(U4-PC4-Pad24) -> Net-(U4-PC4)
- U4 pad 25: unconnected-(U4-PC5-Pad25) -> Net-(U4-PC5)
- U5 pad 2: unconnected-(U5-DIR-Pad2) -> Net-(RN2-R1.2)
- U5 pad 22: unconnected-(U5-~{OE}-Pad22) -> /MCU/HOUR_~{OE}
- U6 pad 2: unconnected-(U6-DIR-Pad2) -> Net-(RN1-R1.2)
- U6 pad 22: unconnected-(U6-~{OE}-Pad22) -> /MCU/MIN_~{OE}
Routing:
- net /MCU/HOUR_~{OE}: track 0.00 -> 58.0 mm, vias 0 -> 2
- net /MCU/MIN_~{OE}: track 0.00 -> 52.1 mm, vias 0 -> 2
- net +3V3: track 298.1 -> 323.1 mm, vias 15 -> 17
- net GND: track 64.3 -> 81.1 mm, vias 464 -> 456
- net Net-(RN1-R1.2): track 0.00 -> 6.77 mm, vias 0 -> 1
- net Net-(U4-PC5): track 0.00 -> 6.56 mm
- net Net-(U4-PC4): track 0.00 -> 6.20 mm
- net Net-(RN2-R1.2): track 0.00 -> 5.85 mm, vias 0 -> 1
- net /MCU/MH_D: track 34.7 -> 29.4 mm
- net /MCU/BTNUP: track 124.7 -> 121.0 mm
- net Net-(F1-Pad1): track 0.00 -> 2.65 mm
- net +100V: track 130.2 -> 132.7 mm
- net /MCU/NRST: track 27.7 -> 25.6 mm
- net /MCU/HL_A: track 45.9 -> 43.9 mm
- net /MCU/MH_C: track 30.6 -> 32.5 mm
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Other:
- board text added: "+"
